File: pcb/hackbar.kicad_sch (KiCad schematic)
At the start: 26 parts, among them SW1 SW_Push, SW2 SW_Push, SW3 SW_Push, SW4 SW_Push, SW5 SW_Push, SW6 SW_Push, SW7 SW_Push, SW8 SW_Push, U1 XIAO-RP2040-SMD

Commit message: pcb layout + final touches + cad
Parts:
- removed D15, D16: SK6812, 2_udu_lib:SK6812MINI-E_fixed, symbol LED:SK6812
- removed SW8: SW_Push, mxfoot:MX-Hotswap-1U, symbol Switch:SW_Push
- U1: footprint 1_udu_lib:XIAO-RP2040-SMD -> 1_udu_lib:XIAO-RP2040-DIP
Connections:
- net IO0: now also SW7.1; no longer SW1.1
- net IO1: now also D1.2 (DIN); no longer MT1.2
- net IO2: no longer SW7.1
- net IO26: now also SW4.1; no longer SW6.1
- net IO27: now also SW3.1; no longer SW5.1
- net IO28: now also SW2.1; no longer D1.2 (DIN)
- net IO29: now also SW1.1; no longer SW4.1
- net IO6: now also SW5.1; no longer SW3.1
- net IO7: now also SW6.1; no longer SW2.1
- net IO3: now reaches U1.11 (GPIO3_D10_MOSI)
- net IO3: now also MT1.2
Other:
- moved on the sheet: MT1, SW1, SW2, SW3, SW4, SW5, SW6, SW7

Commit message: add cad, images, readme, bom
Parts:
- added D15, D16: SK6812, 2_udu_lib:SK6812MINI-E_fixed, symbol LED:SK6812
Connections:
- net +5V: now also D15.3 (VDD), D16.3 (VDD)
- net GND: now also D15.1 (VSS), D16.1 (VSS)
- net IO1: now also D15.2 (DIN); no longer D1.2 (DIN)
- new net: D1.2 (DIN), D16.4 (DOUT)
- new net: D15.4 (DOUT), D16.2 (DIN)
Other:
- moved on the sheet: D1, D10, D11, D12, D13, D14, D2, D3, D4, D5, D6, D7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
